File: KiCad Practice/task_1/task_1.sch (KiCad schematic (older format))
At the start: 47 parts, among them J1 Conn_01x04_Female, J2 USB_OTG, Q1 Q_NMOS_GSD, SW1 SW_Push, U1 XT4052, U2 FS8205A, U3 STM8L051F3P, U4 DW01, U5 MIC5219-2.8YM5

Commit message: stm8L started
Connections:
- net OD: now reaches U2.4 (GATE1)
- net OD: now also U4.1 (OD)
Changed lines of the file:
@@
 Wire Wire Line
 	2500 700  2500 850
+Text Label 3400 6850 2    50   ~ 0
+OD
+Wire Wire Line
+	3450 6850 3400 6850
+Text Label 1400 7100 2    50   ~ 0
+OD
+Wire Wire Line
+	1500 7100 1400 7100
 $EndSCHEMATC
