File: KiCad Practice/task_1/task_1.kicad_pcb (KiCad board)
At the start: 2 copper layers, 50.8 x 50 mm, 47 parts, among them J1 Conn_01x04_Female, J2 USB_OTG, Q1 Q_NMOS_GSD, SW1 SW_Push, U1 XT4052, U2 FS8205A, U3 STM8L051F3P, U4 DW01, U5 MIC5219-2.8YM5

Commit message: stm8L started
Parts:
- moved D2 16.1 mm to (166.9, 61.5)
- moved D4 16.0 mm to (212.9, 62.0)
- moved D6 11.2 mm to (213.0, 108.0)
- moved R14 8.55 mm to (213.1, 65.4)
- moved D5 5.18 mm to (167.6, 108.6)
Connections:
- U2 pad 4: Net-(U2-Pad4) -> /OD
- U4 pad 1: Net-(U4-Pad1) -> /OD
Routing:
- net /3.6V: track 167.4 -> 199.0 mm, vias 2 -> 4
- net Net-(D2-Pad1): track 3.69 -> 20.1 mm
- net /OD: track 0.00 -> 9.81 mm, vias 0 -> 2
- net Net-(Q1-Pad3): track 101.9 -> 110.7 mm
- net Net-(D6-Pad1): track 3.50 -> 11.2 mm
- net Net-(D5-Pad1): track 3.52 -> 8.90 mm
- net Net-(D4-Pad1): track 4.89 -> 4.03 mm
- added copper zone on B.Cu, net GND
- added copper zone on F.Cu, net GND
Other:
- board text added: "-"
- board text added: "2.8V"
- board text added: "GND"
- board text added: "NRST"
- board text added: "SWM"
- board text added: "Stat"
